File: aek.kicad_sch (KiCad schematic)
At the start: 243 parts, among them J1 Conn_01x04_MountingPin, SW1 SW_Push, U1 ATmega32U4-MU, Y1 16MHz

Commit message: push
Parts:
- LED1, LED2, LED3: symbol ws2812b:WS2812B -> random-keyboard-parts:WS2812B
- SW_0, SW_1, SW_2, SW_3, SW_4, SW_5, SW_6, SW_7, SW_8, SW_9, SW_A1, SW_APOS1, SW_B1, SW_BACKSP1, SW_BKSLS1, SW_C1, SW_CAP1, SW_COLON1, SW_COMMA1, SW_D1, SW_DEL1, SW_DOWN1, SW_E1, SW_END1, SW_ENTER1, SW_EQ1, SW_ESC1, SW_F1, SW_F10, SW_F11, SW_F12, SW_F13, SW_F2, SW_F3, SW_F4, SW_F5, SW_F6, SW_F7, SW_F8, SW_F9, SW_G1, SW_H1, SW_HOME1, SW_I1, SW_INS1, SW_J1, SW_K1, SW_KP0, SW_KP0ALT1, SW_KP0X1, SW_KP1, SW_KP2, SW_KP3, SW_KP4, SW_KP5, SW_KP6, SW_KP7, SW_KP8, SW_KP9, SW_KPASTR1, SW_KPENTER1, SW_KPENTERALT1, SW_KPENTERX1, SW_KPEQ1, SW_KPMINUS1, SW_KPPER1, SW_KPPLUS1, SW_KPSLASH1, SW_L1, SW_LALT1, SW_LBRAC1, SW_LCTR1, SW_LEFT1, SW_LMOD1, SW_LSH1, SW_M1, SW_MINUS1, SW_N1, SW_NUMLK1, SW_O1, SW_P1, SW_PAUSE1, SW_PERIOD1, SW_PGDN1, SW_PGUP1, SW_POW1, SW_PRSC1, SW_Q1, SW_R1, SW_RALT1, SW_RBRAC1, SW_RCTR1, SW_RIGHT1, SW_RMOD1, SW_RSH1, SW_S1, SW_SCLK1, SW_SLASH1, SW_SPACE1, SW_T1, SW_TAB1, SW_TICK1, SW_U1, SW_UP1, SW_V1, SW_W1, SW_X1, SW_Y1, SW_Z1: symbol MX_Alps_Hybrid:MX-NoLED -> random-keyboard-parts:MX-NoLED
- U1: footprint atmega32u4-au-and-mu:atmega32u4-mu-and-au -> random-keyboard-parts:atmega32u4-mu-and-au; symbol MCU_Microchip_ATmega:ATmega32U4-MU -> MCU_Microchip_ATmega:ATmega32U4-M
